File: hw/offset_dac.sch (KiCad schematic (older format))
At the start: 27 parts, among them U11 TSV992A, U14 MCP47CVB02-E_UN

Commit message: more work (don't recall details :-()
Parts:
- removed C83, C84: 200p, Capacitor_SMD:C_0603_1608Metric, symbol fmc:100nF_603
- removed R57, R59: 75k, Resistor_SMD:R_0603_1608Metric, symbol Device:R_Small
- R61, R62: value 10 -> 1
- U11: footprint (none) -> Package_SO:MSOP-8_3x3mm_P0.65mm
Connections:
- net GND is gone; now on net GNDA: C78.2, C79.2, C80.2, C81.2
- net at R52.2, R58.2, U11.2 (-): now also C85.2
- net at R54.2, R60.2, U11.6 (-): now also C86.2
Changed lines of the file:
@@
 F 0 "U11" H 6050 2267 50  0000 C CNN
 F 1 "TSV992A" H 6050 2176 50  0000 C CNN
-F 2 "" H 6050 1900 50  0001 C CNN
+F 2 "Package_SO:MSOP-8_3x3mm_P0.65mm" H 6050 1900 50  0001 C CNN
 F 3 "~" H 6050 1900 50  0001 C CNN
 	1    6050 1900
@@
 F 0 "U11" H 6050 4217 50  0000 C CNN
 F 1 "TSV992A" H 6050 4126 50  0000 C CNN
-F 2 "" H 6050 3850 50  0001 C CNN
+F 2 "Package_SO:MSOP-8_3x3mm_P0.65mm" H 6050 3850 50  0001 C CNN
 F 3 "~" H 6050 3850 50  0001 C CNN
 	2    6050 3850
@@
 F 0 "U11" V 1875 2300 50  0000 C CNN
 F 1 "TSV992A" V 1966 2300 50  0000 C CNN
-F 2 "" H 2200 2300 50  0001 C CNN
+F 2 "Package_SO:MSOP-8_3x3mm_P0.65mm" H 2200 2300 50  0001 C CNN
 F 3 "~" H 2200 2300 50  0001 C CNN
 	3    2200 2300
@@
 AR Path="/612B1274/60C14D80/60C291B7" Ref="R61"  Part="1"
 F 0 "R61" V 6804 1900 50  0000 C CNN
-F 1 "10" V 6895 1900 50  0000 C CNN
+F 1 "1" V 6895 1900 50  0000 C CNN
 F 2 "Resistor_SMD:R_0603_1608Metric" H 7000 1900 50  0001 C CNN
 F 3 "~" H 7000 1900 50  0001 C CNN
@@
 Wire Wire Line
 	6350 1900 6800 1900
-$Comp
-L Device:R_Small R?
-U 1 1 60C293AE
-P 6150 2200
-AR Path="/612B1274/60C293AE" Ref="R?"  Part="1"
-AR Path="/612B1274/60C14D80/60C293AE" Ref="R57"  Part="1"
-F 0 "R57" V 5954 2200 50  0000 C CNN
-F 1 "75k" V 6045 2200 50  0000 C CNN
-F 2 "Resistor_SMD:R_0603_1608Metric" H 6150 2200 50  0001 C CNN
-F 3 "~" H 6150 2200 50  0001 C CNN
-	1    6150 2200
-	0    1    1    0
-$EndComp
 Wire Wire Line
 	5750 2000 5750 2200
-Wire Wire Line
-	5750 2200 6050 2200
 $Comp
 L fmc:100nF_603 C?
@@
 Wire Wire Line
 	6800 1900 6900 1900
-Wire Wire Line
-	6350 2200 6250 2200
 $Comp
 L Device:R_Small R?
@@
 	0    1    1    0
 $EndComp
-$Comp
-L fmc:100nF_603 C?
-U 1 1 60C2D7C1
-P 6150 2850
-AR Path="/6086F2E3/60C2D7C1" Ref="C?"  Part="1"
-AR Path="/60B16D71/60C2D7C1" Ref="C?"  Part="1"
-AR Path="/612B1274/60C2D7C1" Ref="C?"  Part="1"
-AR Path="/612B1274/60C14D80/60C2D7C1" Ref="C83"  Part="1"
-F 0 "C83" H 6350 2850 50  0000 C CNN
-F 1 "200p" H 6350 2950 50  0000 C CNN
-F 2 "Capacitor_SMD:C_0603_1608Metric" H 6188 2700 50  0001 C CNN
-F 3 "~" H 6150 2850 50  0001 C CNN
-F 4 "" H 6275 3050 50  0001 C CNN "Part"
-F 5 "Murata" H 6375 3150 50  0001 C CNN "Manufacturer"
-	1    6150 2850
-	0    1    1    0
-$EndComp
 Wire Wire Line
 	6050 2600 5750 2600
@@
 	5750 2600 5750 2200
 Connection ~ 5750 2200
-Wire Wire Line
-	6000 2850 5750 2850
-Wire Wire Line
-	5750 2850 5750 2600
 Connection ~ 5750 2600
 Wire Wire Line
-	6250 2600 6400 2600
-Wire Wire Line
 	7200 2600 7200 1900
 Wire Wire Line
 	7200 1900 7100 1900
-Wire Wire Line
-	6300 2850 6400 2850
-Wire Wire Line
-	6400 2850 6400 2600
-Connection ~ 6400 2600
-Wire Wire Line
-	6400 2600 7200 2600
 $Comp
 L fmc:100nF_603 C?
@@
 AR Path="/612B1274/60C14D80/60C42CEE" Ref="R62"  Part="1"
 F 0 "R62" V 6804 3850 50  0000 C CNN
-F 1 "10" V 6895 3850 50  0000 C CNN
+F 1 "1" V 6895 3850 50  0000 C CNN
 F 2 "Resistor_SMD:R_0603_1608Metric" H 7000 3850 50  0001 C CNN
 F 3 "~" H 7000 3850 50  0001 C CNN
@@
 Wire Wire Line
 	6350 3850 6800 3850
-$Comp
-L Device:R_Small R?
-U 1 1 60C42CF9
-P 6150 4150
-AR Path="/612B1274/60C42CF9" Ref="R?"  Part="1"
-AR Path="/612B1274/60C14D80/60C42CF9" Ref="R59"  Part="1"
-F 0 "R59" V 5954 4150 50  0000 C CNN
-F 1 "75k" V 6045 4150 50  0000 C CNN
-F 2 "Resistor_SMD:R_0603_1608Metric" H 6150 4150 50  0001 C CNN
-F 3 "~" H 6150 4150 50  0001 C CNN
-	1    6150 4150
-	0    1    1    0
-$EndComp
 Wire Wire Line
 	5750 3950 5750 4150
-Wire Wire Line
-	5750 4150 6050 4150
 $Comp
 L fmc:100nF_603 C?
@@
 Wire Wire Line
 	6800 3850 6900 3850
-Wire Wire Line
-	6350 4150 6250 4150
 $Comp
 L Device:R_Small R?
@@
 	0    1    1    0
 $EndComp
-$Comp
-L fmc:100nF_603 C?
-U 1 1 60C42D22
-P 6150 4800
-AR Path="/6086F2E3/60C42D22" Ref="C?"  Part="1"
-AR Path="/60B16D71/60C42D22" Ref="C?"  Part="1"
-AR Path="/612B1274/60C42D22" Ref="C?"  Part="1"
-AR Path="/612B1274/60C14D80/60C42D22" Ref="C84"  Part="1"
-F 0 "C84" H 6350 4800 50  0000 C CNN
-F 1 "200p" H 6350 4900 50  0000 C CNN
-F 2 "Capacitor_SMD:C_0603_1608Metric" H 6188 4650 50  0001 C CNN
-F 3 "~" H 6150 4800 50  0001 C CNN
-F 4 "" H 6275 5000 50  0001 C CNN "Part"
-F 5 "Murata" H 6375 5100 50  0001 C CNN "Manufacturer"
-	1    6150 4800
-	0    1    1    0
-$EndComp
 Wire Wire Line
 	6050 4550 5750 4550
@@
 	5750 4550 5750 4150
 Connection ~ 5750 4150
-Wire Wire Line
-	6000 4800 5750 4800
-Wire Wire Line
-	5750 4800 5750 4550
 Connection ~ 5750 4550
 Wire Wire Line
-	6250 4550 6400 4550
-Wire Wire Line
 	7200 4550 7200 3850
 Wire Wire Line
 	7200 3850 7100 3850
-Wire Wire Line
-	6300 4800 6400 4800
-Wire Wire Line
-	6400 4800 6400 4550
-Connection ~ 6400 4550
-Wire Wire Line
-	6400 4550 7200 4550
 $Comp
 L fmc:100nF_603 C?
@@
 	-1   0    0    1
 $EndComp
-$Comp
-L power:GND #PWR?
-U 1 1 60C51CDF
-P 2900 2500
-AR Path="/6086F2E3/60C51CDF" Ref="#PWR?"  Part="1"
-AR Path="/60AABC24/60C51CDF" Ref="#PWR?"  Part="1"
-AR Path="/60B16D71/60C51CDF" Ref="#PWR?"  Part="1"
-AR Path="/612B1274/60C51CDF" Ref="#PWR?"  Part="1"
-AR Path="/612B1274/611783BC/60C51CDF" Ref="#PWR?"  Part="1"
-AR Path="/612B1274/611E90A8/60C51CDF" Ref="#PWR?"  Part="1"
-AR Path="/612B1274/60C14D80/60C51CDF" Ref="#PWR?"  Part="1"
-F 0 "#PWR?" H 2900 2250 50  0001 C CNN
-F 1 "GND" H 2905 2327 50  0000 C CNN
-F 2 "" H 2900 2500 50  0001 C CNN
-F 3 "" H 2900 2500 50  0001 C CNN
-	1    2900 2500
-	1    0    0    -1
-$EndComp
 Wire Wire Line
 	2900 2500 3050 2500
@@
 	1    0    0    -1
 $EndComp
-$Comp
-L power:GND #PWR?
-U 1 1 60C51D09
-P 1100 2500
-AR Path="/6086F2E3/60C51D09" Ref="#PWR?"  Part="1"
-AR Path="/60AABC24/60C51D09" Ref="#PWR?"  Part="1"
-AR Path="/60B16D71/60C51D09" Ref="#PWR?"  Part="1"
-AR Path="/612B1274/60C51D09" Ref="#PWR?"  Part="1"
-AR Path="/612B1274/611783BC/60C51D09" Ref="#PWR?"  Part="1"
-AR Path="/612B1274/611E90A8/60C51D09" Ref="#PWR?"  Part="1"
-AR Path="/612B1274/60C14D80/60C51D09" Ref="#PWR?"  Part="1"
-F 0 "#PWR?" H 1100 2250 50  0001 C CNN
-F 1 "GND" H 1105 2327 50  0000 C CNN
-F 2 "" H 1100 2500 50  0001 C CNN
-F 3 "" H 1100 2500 50  0001 C CNN
-	1    1100 2500
-	1    0    0    -1
-$EndComp
 Wire Wire Line
 	1100 2500 1250 2500
@@
 	8650 1900 7950 1900
 Connection ~ 7950 1900
+Wire Wire Line
+	6250 4550 7200 4550
+Wire Wire Line
+	6250 2600 7200 2600
+Wire Wire Line
+	5750 4150 6350 4150
+Wire Wire Line
+	5750 2200 6350 2200
+$Comp
+L power:GNDA #PWR?
+U 1 1 60D0F45C
+P 2900 2500
+AR Path="/612B1274/60D0F45C" Ref="#PWR?"  Part="1"
+AR Path="/612B1274/60C14D80/60D0F45C" Ref="#PWR?"  Part="1"
+F 0 "#PWR?" H 2900 2250 50  0001 C CNN
+F 1 "GNDA" H 2905 2327 50  0000 C CNN
+F 2 "" H 2900 2500 50  0001 C CNN
+F 3 "" H 2900 2500 50  0001 C CNN
+	1    2900 2500
+	1    0    0    -1
+$EndComp
+$Comp
+L power:GNDA #PWR?
+U 1 1 60D0F8C3
+P 1100 2500
+AR Path="/612B1274/60D0F8C3" Ref="#PWR?"  Part="1"
+AR Path="/612B1274/60C14D80/60D0F8C3" Ref="#PWR?"  Part="1"
+F 0 "#PWR?" H 1100 2250 50  0001 C CNN
+F 1 "GNDA" H 1105 2327 50  0000 C CNN
+F 2 "" H 1100 2500 50  0001 C CNN
+F 3 "" H 1100 2500 50  0001 C CNN
+	1    1100 2500
+	1    0    0    -1
+$EndComp
 $EndSCHEMATC

Commit message: everything hooked up + layed out; 0.2/0.4mm vias :-(
Parts:
- U11: footprint Package_SO:MSOP-8_3x3mm_P0.65mm -> proj_footprints:DFN-8-1EP_2x2mm_P0.5mm_EP0.45x1.6mm
Changed lines of the file:
@@
 $Descr A4 11693 8268
 encoding utf-8
-Sheet 8 8
+Sheet 9 9
 Title ""
 Date ""
@@
 F 0 "U11" H 6050 2267 50  0000 C CNN
 F 1 "TSV992A" H 6050 2176 50  0000 C CNN
-F 2 "Package_SO:MSOP-8_3x3mm_P0.65mm" H 6050 1900 50  0001 C CNN
+F 2 "proj_footprints:DFN-8-1EP_2x2mm_P0.5mm_EP0.45x1.6mm" H 6050 1900 50  0001 C CNN
 F 3 "~" H 6050 1900 50  0001 C CNN
 	1    6050 1900
@@
 F 0 "U11" H 6050 4217 50  0000 C CNN
 F 1 "TSV992A" H 6050 4126 50  0000 C CNN
-F 2 "Package_SO:MSOP-8_3x3mm_P0.65mm" H 6050 3850 50  0001 C CNN
+F 2 "proj_footprints:DFN-8-1EP_2x2mm_P0.5mm_EP0.45x1.6mm" H 6050 3850 50  0001 C CNN
 F 3 "~" H 6050 3850 50  0001 C CNN
 	2    6050 3850
@@
 F 0 "U11" V 1875 2300 50  0000 C CNN
 F 1 "TSV992A" V 1966 2300 50  0000 C CNN
-F 2 "Package_SO:MSOP-8_3x3mm_P0.65mm" H 2200 2300 50  0001 C CNN
+F 2 "proj_footprints:DFN-8-1EP_2x2mm_P0.5mm_EP0.45x1.6mm" H 2200 2300 50  0001 C CNN
 F 3 "~" H 2200 2300 50  0001 C CNN
 	3    2200 2300
