File: hw/buffer.sch (KiCad schematic (older format))
At the start: 13 parts, among them J6 BNC, U12 OPA859xDSG

Commit message: prototype version
Changed lines of the file:
@@
 AR Path="/612B1274/611783BC/61178C80" Ref="U12"  Part="1"
 AR Path="/612B1274/611E90A8/61178C80" Ref="U13"  Part="1"
-F 0 "U12" H 6500 3200 50  0000 C CNN
+F 0 "U13" H 6500 3200 50  0000 C CNN
 F 1 "OPA859xDSG" H 6700 3100 50  0000 C CNN
 F 2 "Package_SON:WSON-8-1EP_2x2mm_P0.5mm_EP0.9x1.6mm" H 6250 4000 50  0001 C CNN
@@
 AR Path="/612B1274/611783BC/611A4FDB" Ref="J6"  Part="1"
 AR Path="/612B1274/611E90A8/611A4FDB" Ref="J8"  Part="1"
-F 0 "J6" H 3650 3475 50  0000 L CNN
+F 0 "J8" H 3650 3475 50  0000 L CNN
 F 1 "BNC" H 3650 3384 50  0000 L CNN
 F 2 "proj_footprints:BNC_Molex_0731713150" H 3550 3500 50  0001 C CNN
@@
 AR Path="/612B1274/611783BC/611A70F5" Ref="R47"  Part="1"
 AR Path="/612B1274/611E90A8/611A70F5" Ref="R49"  Part="1"
-F 0 "R47" V 3954 3500 50  0000 C CNN
+F 0 "R49" V 3954 3500 50  0000 C CNN
 F 1 "500k" V 4045 3500 50  0000 C CNN
 F 2 "Resistor_SMD:R_0603_1608Metric" H 4150 3500 50  0001 C CNN
@@
 AR Path="/612B1274/611783BC/611D1DE7" Ref="C70"  Part="1"
 AR Path="/612B1274/611E90A8/611D1DE7" Ref="C76"  Part="1"
-F 0 "C70" H 7450 5200 50  0000 L CNN
+F 0 "C76" H 7450 5200 50  0000 L CNN
 F 1 "100n" H 7400 4700 50  0000 L CNN
 F 2 "Capacitor_SMD:C_0402_1005Metric" H 7438 4800 50  0001 C CNN
@@
 AR Path="/612B1274/611783BC/611D4AAD" Ref="C71"  Part="1"
 AR Path="/612B1274/611E90A8/611D4AAD" Ref="C77"  Part="1"
-F 0 "C71" H 7650 5200 50  0000 L CNN
+F 0 "C77" H 7650 5200 50  0000 L CNN
 F 1 "1u" H 7650 4700 50  0000 L CNN
 F 2 "Capacitor_SMD:C_0805_2012Metric" H 7738 4800 50  0001 C CNN
@@
 AR Path="/612B1274/611783BC/611D5312" Ref="C68"  Part="1"
 AR Path="/612B1274/611E90A8/611D5312" Ref="C74"  Part="1"
-F 0 "C68" H 5650 5250 50  0000 L CNN
+F 0 "C74" H 5650 5250 50  0000 L CNN
 F 1 "100n" H 5600 4750 50  0000 L CNN
 F 2 "Capacitor_SMD:C_0402_1005Metric" H 5638 4850 50  0001 C CNN
@@
 AR Path="/612B1274/611783BC/611D532F" Ref="C69"  Part="1"
 AR Path="/612B1274/611E90A8/611D532F" Ref="C75"  Part="1"
-F 0 "C69" H 5850 5250 50  0000 L CNN
+F 0 "C75" H 5850 5250 50  0000 L CNN
 F 1 "1u" H 5850 4750 50  0000 L CNN
 F 2 "Capacitor_SMD:C_0805_2012Metric" H 5938 4850 50  0001 C CNN
@@
 AR Path="/612B1274/611783BC/61207E57" Ref="C67"  Part="1"
 AR Path="/612B1274/611E90A8/61207E57" Ref="C73"  Part="1"
-F 0 "C67" H 5150 3650 50  0000 C CNN
+F 0 "C73" H 5150 3650 50  0000 C CNN
 F 1 "15p" H 5150 3750 50  0000 C CNN
 F 2 "Capacitor_SMD:C_0603_1608Metric" H 4988 3500 50  0001 C CNN
@@
 AR Path="/612B1274/611783BC/61208FD0" Ref="C66"  Part="1"
 AR Path="/612B1274/611E90A8/61208FD0" Ref="C72"  Part="1"
-F 0 "C66" H 4350 3150 50  0000 C CNN
+F 0 "C72" H 4350 3150 50  0000 C CNN
 F 1 "20p" H 4350 3250 50  0000 C CNN
 F 2 "Capacitor_SMD:C_0603_1608Metric" H 4188 3000 50  0001 C CNN
@@
 AR Path="/612B1274/611783BC/611A713B" Ref="R48"  Part="1"
 AR Path="/612B1274/611E90A8/611A713B" Ref="R50"  Part="1"
-F 0 "R48" V 4304 3650 50  0000 C CNN
+F 0 "R50" V 4304 3650 50  0000 C CNN
 F 1 "500k" V 4395 3650 50  0000 C CNN
 F 2 "Resistor_SMD:R_0603_1608Metric" H 4500 3650 50  0001 C CNN
@@
 AR Path="/612B1274/611783BC/60D14E8F" Ref="C98"  Part="1"
 AR Path="/612B1274/611E90A8/60D14E8F" Ref="C99"  Part="1"
-F 0 "C98" H 5441 3696 50  0000 L CNN
+F 0 "C99" H 5441 3696 50  0000 L CNN
 F 1 "5-15p" H 5441 3605 50  0000 L CNN
 F 2 "proj_footprints:C_Trimmer_EW_Electronics_SCG3S" H 5350 3650 50  0001 C CNN
@@
 AR Path="/612B1274/611E90A8/60F53174" Ref="R82"  Part="1"
 AR Path="/612B1274/611783BC/60F53174" Ref="R80"  Part="1"
-F 0 "R80" V 5854 2900 50  0000 C CNN
+F 0 "R82" V 5854 2900 50  0000 C CNN
 F 1 "750" V 5945 2900 50  0000 C CNN
 F 2 "Resistor_SMD:R_0402_1005Metric" H 6050 2900 50  0001 C CNN
@@
 AR Path="/612B1274/611E90A8/60F5371A" Ref="R81"  Part="1"
 AR Path="/612B1274/611783BC/60F5371A" Ref="R79"  Part="1"
-F 0 "R79" V 5354 2900 50  0000 C CNN
+F 0 "R81" V 5354 2900 50  0000 C CNN
 F 1 "150" V 5445 2900 50  0000 C CNN
 F 2 "Resistor_SMD:R_0402_1005Metric" H 5550 2900 50  0001 C CNN
