File: hw/digio.sch (KiCad schematic (older format))
At the start: 11 parts, among them J2001 BNC, U17 SN74LVC2T45DCUR

Commit message: prototype version
Connections:
- net +1V8: no longer R2001.1, U17.1 (VCCA)
- net DIGIO: now reaches D13.2 (A), D14.1 (K), R2004.1, R2005.1, U17.6 (B2), U17.7 (B1)
- new net VCC_LOGIC: R2001.1, U17.1 (VCCA)
Other:
- moved on the sheet: D13, D14, J10, R77, R78
Changed lines of the file:
@@
 L Device:R_Small R?
 U 1 1 60F26603
-P 6900 4150
+P 7650 4150
 AR Path="/60DC28BD/60F26603" Ref="R?"  Part="1"
 AR Path="/60F26603" Ref="R?"  Part="1"
@@
 AR Path="/60F0CD00/60F26603" Ref="R77"  Part="1"
 AR Path="/60AABC24/60F79994/60F26603" Ref="R78"  Part="1"
-F 0 "R78" H 6959 4196 50  0000 L CNN
-F 1 "50" H 6959 4105 50  0000 L CNN
-F 2 "Resistor_SMD:R_0603_1608Metric" H 6900 4150 50  0001 C CNN
-F 3 "~" H 6900 4150 50  0001 C CNN
-	1    6900 4150
+F 0 "R78" H 7709 4196 50  0000 L CNN
+F 1 "50" H 7709 4105 50  0000 L CNN
+F 2 "Resistor_SMD:R_0603_1608Metric" H 7650 4150 50  0001 C CNN
+F 3 "~" H 7650 4150 50  0001 C CNN
+	1    7650 4150
 	0    -1   -1   0
 $EndComp
@@
 L Connector:Conn_Coaxial J?
 U 1 1 60E51E93
-P 7650 4150
+P 8400 4150
 AR Path="/60B16D71/60E51E93" Ref="J?"  Part="1"
 AR Path="/612B1274/60E51E93" Ref="J?"  Part="1"
@@
 AR Path="/60F0CD00/60E51E93" Ref="J10"  Part="1"
 AR Path="/60AABC24/60F79994/60E51E93" Ref="J10"  Part="1"
-F 0 "J10" H 7750 4125 50  0000 L CNN
-F 1 "BNC" H 7750 4034 50  0000 L CNN
-F 2 "proj_footprints:BNC_Molex_0731713150" H 7650 4150 50  0001 C CNN
-F 3 " ~" H 7650 4150 50  0001 C CNN
-F 4 "0731713150" H 7650 4150 50  0001 C CNN "Part"
-F 5 "Molex" H 7650 4150 50  0001 C CNN "Manufacturer"
-	1    7650 4150
+F 0 "J10" H 8500 4125 50  0000 L CNN
+F 1 "BNC" H 8500 4034 50  0000 L CNN
+F 2 "proj_footprints:BNC_Molex_0731713150" H 8400 4150 50  0001 C CNN
+F 3 " ~" H 8400 4150 50  0001 C CNN
+F 4 "0731713150" H 8400 4150 50  0001 C CNN "Part"
+F 5 "Molex" H 8400 4150 50  0001 C CNN "Manufacturer"
+	1    8400 4150
 	1    0    0    -1
 $EndComp
@@
 L Device:R_Small R?
 U 1 1 60F05839
-P 6650 4500
+P 7400 4500
 AR Path="/60DC28BD/60F05839" Ref="R?"  Part="1"
 AR Path="/60F05839" Ref="R?"  Part="1"
@@
 AR Path="/60F0CD00/60F05839" Ref="R78"  Part="1"
 AR Path="/60AABC24/60F79994/60F05839" Ref="R77"  Part="1"
-F 0 "R77" H 6709 4546 50  0000 L CNN
-F 1 "100k" H 6709 4455 50  0000 L CNN
-F 2 "Resistor_SMD:R_0603_1608Metric" H 6650 4500 50  0001 C CNN
-F 3 "~" H 6650 4500 50  0001 C CNN
-	1    6650 4500
+F 0 "R77" H 7459 4546 50  0000 L CNN
+F 1 "100k" H 7459 4455 50  0000 L CNN
+F 2 "Resistor_SMD:R_0603_1608Metric" H 7400 4500 50  0001 C CNN
+F 3 "~" H 7400 4500 50  0001 C CNN
+	1    7400 4500
 	1    0    0    -1
 $EndComp
@@
 Wire Wire Line
 	5750 4050 5800 4050
-Wire Wire Line
-	5250 3550 5250 3600
 Wire Wire Line
 	5350 4650 5350 4850
@@
 L power:GND #PWR?
 U 1 1 60F26CE8
-P 7650 4500
+P 8400 4500
 AR Path="/6086F2E3/60F26CE8" Ref="#PWR?"  Part="1"
 AR Path="/60AABC24/60F26CE8" Ref="#PWR?"  Part="1"
 AR Path="/60F0CD00/60F26CE8" Ref="#PWR?"  Part="1"
 AR Path="/60AABC24/60F79994/60F26CE8" Ref="#PWR?"  Part="1"
-F 0 "#PWR?" H 7650 4250 50  0001 C CNN
-F 1 "GND" H 7655 4327 50  0000 C CNN
-F 2 "" H 7650 4500 50  0001 C CNN
-F 3 "" H 7650 4500 50  0001 C CNN
-	1    7650 4500
+F 0 "#PWR?" H 8400 4250 50  0001 C CNN
+F 1 "GND" H 8405 4327 50  0000 C CNN
+F 2 "" H 8400 4500 50  0001 C CNN
+F 3 "" H 8400 4500 50  0001 C CNN
+	1    8400 4500
 	1    0    0    -1
 $EndComp
@@
 $Comp
 L power:+1V8 #PWR?
-U 1 1 60F3DEA2
-P 5250 3550
-AR Path="/6086F2E3/60F3DEA2" Ref="#PWR?"  Part="1"
-AR Path="/60F0CD00/60F3DEA2" Ref="#PWR?"  Part="1"
-AR Path="/60AABC24/60F79994/60F3DEA2" Ref="#PWR?"  Part="1"
-F 0 "#PWR?" H 5250 3400 50  0001 C CNN
-F 1 "+1V8" H 5265 3723 50  0000 C CNN
-F 2 "" H 5250 3550 50  0001 C CNN
-F 3 "" H 5250 3550 50  0001 C CNN
-	1    5250 3550
-	1    0    0    -1
-$EndComp
-$Comp
-L power:+1V8 #PWR?
 U 1 1 60F3E5CB
 P 9350 4550
@@
 Wire Wire Line
 	4500 2400 5450 2400
-Wire Wire Line
-	5450 2400 5450 3600
 $Comp
 L Device:D_Schottky_Small D?
 U 1 1 60F6B1B6
-P 6200 4500
+P 6950 4500
 AR Path="/612B1274/60F6B1B6" Ref="D?"  Part="1"
 AR Path="/60F0CD00/60F6B1B6" Ref="D14"  Part="1"
 AR Path="/60AABC24/60F79994/60F6B1B6" Ref="D14"  Part="1"
-F 0 "D14" V 6154 4570 50  0000 L CNN
-F 1 "NSR0170HT1G" V 7150 4050 50  0001 L CNN
-F 2 "Diode_SMD:D_SOD-323" V 6200 4500 50  0001 C CNN
-F 3 "~" V 6200 4500 50  0001 C CNN
-F 4 "NSR0170HT1G" V 6200 4500 50  0001 C CNN "Part"
-F 5 "OnSemi" V 6200 4500 50  0001 C CNN "Manufacturer"
-	1    6200 4500
+F 0 "D14" V 6904 4570 50  0000 L CNN
+F 1 "NSR0170HT1G" V 7900 4050 50  0001 L CNN
+F 2 "Diode_SMD:D_SOD-323" V 6950 4500 50  0001 C CNN
+F 3 "~" V 6950 4500 50  0001 C CNN
+F 4 "NSR0170HT1G" V 6950 4500 50  0001 C CNN "Part"
+F 5 "OnSemi" V 6950 4500 50  0001 C CNN "Manufacturer"
+	1    6950 4500
 	0    1    1    0
 $EndComp
-Wire Wire Line
-	5800 4050 5800 4150
 $Comp
 L Device:D_Schottky_Small D?
 U 1 1 60F6CE22
-P 6200 3850
+P 6950 3850
 AR Path="/612B1274/60F6CE22" Ref="D?"  Part="1"
 AR Path="/60F0CD00/60F6CE22" Ref="D13"  Part="1"
 AR Path="/60AABC24/60F79994/60F6CE22" Ref="D13"  Part="1"
-F 0 "D13" V 6154 3920 50  0000 L CNN
-F 1 "NSR0170HT1G" V 7150 3400 50  0001 L CNN
-F 2 "Diode_SMD:D_SOD-323" V 6200 3850 50  0001 C CNN
-F 3 "~" V 6200 3850 50  0001 C CNN
-F 4 "NSR0170HT1G" V 6200 3850 50  0001 C CNN "Part"
-F 5 "OnSemi" V 6200 3850 50  0001 C CNN "Manufacturer"
-	1    6200 3850
+F 0 "D13" V 6904 3920 50  0000 L CNN
+F 1 "NSR0170HT1G" V 7900 3400 50  0001 L CNN
+F 2 "Diode_SMD:D_SOD-323" V 6950 3850 50  0001 C CNN
+F 3 "~" V 6950 3850 50  0001 C CNN
+F 4 "NSR0170HT1G" V 6950 3850 50  0001 C CNN "Part"
+F 5 "OnSemi" V 6950 3850 50  0001 C CNN "Manufacturer"
+	1    6950 3850
 	0    1    1    0
 $EndComp
 Wire Wire Line
-	5800 4150 6200 4150
-Connection ~ 5800 4150
-Wire Wire Line
-	5800 4150 5800 4250
-Wire Wire Line
-	6200 3950 6200 4150
-Connection ~ 6200 4150
-Wire Wire Line
-	6200 4150 6650 4150
-Wire Wire Line
-	6200 4150 6200 4400
-Wire Wire Line
-	5450 3600 6200 3600
-Wire Wire Line
-	6200 3600 6200 3750
-Connection ~ 5450 3600
-Wire Wire Line
-	5450 3600 5450 3650
-Wire Wire Line
-	5350 4850 6200 4850
-Wire Wire Line
-	6200 4850 6200 4600
-Wire Wire Line
-	7000 4150 7450 4150
-Wire Wire Line
-	6650 4400 6650 4150
-Connection ~ 6650 4150
-Wire Wire Line
-	6650 4150 6800 4150
-Wire Wire Line
-	7650 4350 7650 4500
-Wire Wire Line
-	6650 4600 6650 4850
-Wire Wire Line
-	6650 4850 6200 4850
-Connection ~ 6200 4850
+	6950 3950 6950 4150
+Connection ~ 6950 4150
+Wire Wire Line
+	6950 4150 7400 4150
+Wire Wire Line
+	6950 4150 6950 4400
+Wire Wire Line
+	6950 3600 6950 3750
+Wire Wire Line
+	6950 4850 6950 4600
+Wire Wire Line
+	7750 4150 8200 4150
+Wire Wire Line
+	7400 4400 7400 4150
+Connection ~ 7400 4150
+Wire Wire Line
+	7400 4150 7550 4150
+Wire Wire Line
+	8400 4350 8400 4500
+Wire Wire Line
+	7400 4600 7400 4850
+Wire Wire Line
+	7400 4850 6950 4850
+Connection ~ 6950 4850
 Wire Wire Line
 	4100 4150 4200 4150
@@
 Wire Wire Line
 	4550 3600 5250 3600
+Wire Wire Line
+	5450 2400 5450 3600
+Wire Wire Line
+	5800 4050 5800 4150
+Wire Wire Line
+	5450 3600 6950 3600
+Connection ~ 5450 3600
+Wire Wire Line
+	5450 3600 5450 3650
+Wire Wire Line
+	5350 4850 6950 4850
+Wire Wire Line
+	5800 4150 6950 4150
+Connection ~ 5800 4150
+Wire Wire Line
+	5800 4150 5800 4250
+Text Label 6000 4150 0    50   ~ 0
+DIGIO
+Text HLabel 4100 3350 0    50   Input ~ 0
+VCC_LOGIC
+Wire Wire Line
+	4100 3350 5250 3350
+Wire Wire Line
+	5250 3350 5250 3600
 $EndSCHEMATC
