File: hw/fpga_xc3s.sch (KiCad schematic (older format))
At the start: 45 parts, among them J4 JTAG, J5 GPIO_2V5, J6 GPIO_1V8, J9 Conn_02x04_Odd_Even, U5 XC3S50A-VQ100, U6 AT25DF041B

Commit message: several updates...
Parts:
- removed J6: GPIO_1V8, Connector_PinHeader_2.54mm:PinHeader_2x08_P2.54mm_Vertical, symbol Connector_Generic:Conn_02x08_Odd_Even
Connections:
- net labels added: ADC_CSb, ADC_D0, ADC_D1, ADC_D2, ADC_D3, ADC_D4, ADC_D5, ADC_D6, ADC_D7, ADC_DCLK, ADC_DOR, ADC_SCLK, ADC_SDIO, ADC_SYNC
- wire segments 291 -> 263
- no-connect marks 13 -> 9
Changed lines of the file:
@@
 $Descr A4 11693 8268
 encoding utf-8
-Sheet 3 4
+Sheet 3 5
 Title ""
 Date ""
@@
 	7150 3600 7200 3600
 Wire Wire Line
-	7150 3200 7500 3200
-Wire Wire Line
 	7150 2500 7200 2500
 Wire Wire Line
@@
 L power:+1V8 #PWR?
 U 1 1 60B1CE47
-P 7500 3200
+P 8100 3100
 AR Path="/6086F2E3/60B1CE47" Ref="#PWR?"  Part="1"
 AR Path="/60AABC24/60B1CE47" Ref="#PWR?"  Part="1"
-F 0 "#PWR?" H 7500 3050 50  0001 C CNN
-F 1 "+1V8" V 7515 3328 50  0000 L CNN
-F 2 "" H 7500 3200 50  0001 C CNN
-F 3 "" H 7500 3200 50  0001 C CNN
-	1    7500 3200
-	0    1    1    0
-$EndComp
-Wire Wire Line
-	7550 2600 7150 2600
-Wire Wire Line
-	7550 2700 7150 2700
-Wire Wire Line
-	7550 2800 7150 2800
-Wire Wire Line
-	7550 2900 7150 2900
-Wire Wire Line
-	7550 3100 7150 3100
+F 0 "#PWR?" H 8100 2950 50  0001 C CNN
+F 1 "+1V8" V 8115 3228 50  0000 L CNN
+F 2 "" H 8100 3100 50  0001 C CNN
+F 3 "" H 8100 3100 50  0001 C CNN
+	1    8100 3100
+	1    0    0    -1
+$EndComp
 $Comp
 L Memory_Flash:SST25VF080B-50-4x-S2Ax U6
@@
 Wire Wire Line
 	5200 6350 3550 6350
-Text GLabel 5250 1150 1    50   Input ~ 0
+Text GLabel 4550 1150 1    50   Input ~ 0
 FIFO_CLK
-Text GLabel 7550 3500 2    50   BiDi ~ 0
-FIFO_D7
-Text GLabel 7550 3800 2    50   BiDi ~ 0
-FIFO_D6
-Text GLabel 7550 3700 2    50   BiDi ~ 0
-FIFO_D5
-Text GLabel 7550 3100 2    50   BiDi ~ 0
-FIFO_D2
-Text GLabel 7550 3400 2    50   BiDi ~ 0
-FIFO_D1
-Text GLabel 7550 2700 2    50   Input ~ 0
-FIFO_RXE
-Text GLabel 7550 2900 2    50   Input ~ 0
-FIFO_TXF
-Text GLabel 7550 4200 2    50   Output ~ 0
-FIFO_RDb
-Text GLabel 7550 4300 2    50   Output ~ 0
-FIFO_WRb
-Text GLabel 7550 4000 2    50   Output ~ 0
-FIFO_SIWU
-Text GLabel 7550 3900 2    50   BiDi ~ 0
-FIFO_D3
-Text GLabel 7550 2800 2    50   BiDi ~ 0
-FIFO_D4
-Text GLabel 7550 2600 2    50   BiDi ~ 0
-FIFO_D0
-Wire Wire Line
-	7150 3400 7550 3400
-Wire Wire Line
-	7150 3500 7550 3500
-Wire Wire Line
-	7150 3700 7550 3700
-Wire Wire Line
-	7550 3800 7150 3800
-Wire Wire Line
-	7150 3900 7550 3900
-Wire Wire Line
-	7550 4000 7150 4000
-Wire Wire Line
-	7150 4200 7550 4200
-Wire Wire Line
-	7550 4300 7150 4300
 NoConn ~ 7150 4700
 Wire Wire Line
@@
 	0    1    -1   0
 $EndComp
-$Comp
-L fmc:XC3S50A-VQ100 U5
-U 1 1 60AE5529
-P 1650 3000
-F 0 "U5" H 2800 4100 60  0000 L CNN
-F 1 "XC3S50A-VQ100" H 4350 1800 60  0000 L CNN
-F 2 "Package_QFP:VQFP-100_14x14mm_P0.5mm" H 2500 3650 60  0001 R CNN
-F 3 "" H 2500 3450 60  0001 R CNN
-	1    1650 3000
-	1    0    0    -1
-$EndComp
 Wire Wire Line
 	5850 7350 5750 7350
@@
 Wire Wire Line
 	5850 6650 5850 6750
-NoConn ~ 5350 1800
 NoConn ~ 2350 4400
+Text GLabel 4150 1150 1    50   BiDi ~ 0
+I2C_SCL
 Text GLabel 4250 1150 1    50   BiDi ~ 0
-I2C_SCL
-Text GLabel 4150 1150 1    50   BiDi ~ 0
 I2C_SDA
 Wire Wire Line
 	4150 1150 4150 1800
-Text GLabel 4550 1150 1    50   Input ~ 0
+Text GLabel 5150 1150 1    50   Input ~ 0
 FPGA_CLK
 Wire Wire Line
 	4550 1150 4550 1800
 Wire Wire Line
-	5250 1150 5250 1800
-$Comp
-L Connector_Generic:Conn_02x08_Odd_Even J6
-U 1 1 60B60771
-P 1750 3950
-F 0 "J6" V 1754 4330 50  0000 L CNN
-F 1 "GPIO_1V8" V 2250 3750 50  0000 L CNN
-F 2 "Connector_PinHeader_2.54mm:PinHeader_2x08_P2.54mm_Vertical" H 1750 3950 50  0001 C CNN
-F 3 "~" H 1750 3950 50  0001 C CNN
-	1    1750 3950
-	-1   0    0    1
-$EndComp
-Wire Wire Line
-	1950 4250 2350 4250
-Wire Wire Line
-	2350 4250 2350 4300
-Wire Wire Line
-	1950 4150 2250 4150
-Wire Wire Line
-	2250 4150 2250 4200
-Wire Wire Line
-	2250 4200 2350 4200
-Wire Wire Line
-	1950 4050 2250 4050
-Wire Wire Line
-	2250 4050 2250 3900
-Wire Wire Line
-	2250 3900 2350 3900
-Wire Wire Line
-	1950 3950 2150 3950
-Wire Wire Line
-	2150 3950 2150 3800
-Wire Wire Line
-	2150 3800 2350 3800
-Wire Wire Line
-	1950 3850 2250 3850
-Wire Wire Line
-	2250 3850 2250 3600
-Wire Wire Line
-	2250 3600 2350 3600
-Wire Wire Line
-	1950 3750 2150 3750
-Wire Wire Line
-	2150 3750 2150 3500
-Wire Wire Line
-	2150 3500 2350 3500
-Wire Wire Line
-	1300 3400 1350 3400
-Wire Wire Line
-	1950 3650 2100 3650
-Wire Wire Line
-	2100 3650 2100 3300
-Wire Wire Line
-	2100 3300 2350 3300
-Wire Wire Line
-	1950 3550 2000 3550
-Wire Wire Line
-	2000 3550 2000 3200
-Wire Wire Line
-	2000 3200 2350 3200
-Wire Wire Line
-	1450 3550 1400 3550
-Wire Wire Line
-	1400 3550 1400 3750
-$Comp
-L power:GND #PWR?
-U 1 1 60BE2000
-P 1400 4400
-AR Path="/6086F2E3/60BE2000" Ref="#PWR?"  Part="1"
-AR Path="/60AABC24/60BE2000" Ref="#PWR?"  Part="1"
-F 0 "#PWR?" H 1400 4150 50  0001 C CNN
-F 1 "GND" H 1405 4227 50  0000 C CNN
-F 2 "" H 1400 4400 50  0001 C CNN
-F 3 "" H 1400 4400 50  0001 C CNN
-	1    1400 4400
-	1    0    0    -1
-$EndComp
-Wire Wire Line
-	1400 3750 1450 3750
-Connection ~ 1400 3750
-Wire Wire Line
-	1400 3750 1400 3950
-Wire Wire Line
-	1400 3950 1450 3950
-Connection ~ 1400 3950
-Wire Wire Line
-	1400 3950 1400 4150
-Wire Wire Line
-	1400 4150 1450 4150
-Connection ~ 1400 4150
-Wire Wire Line
-	1400 4150 1400 4400
-Wire Wire Line
-	1350 3400 1350 3650
-Wire Wire Line
-	1350 4250 1450 4250
-Connection ~ 1350 3400
-Wire Wire Line
-	1350 3400 2350 3400
-Wire Wire Line
-	1350 4050 1450 4050
-Connection ~ 1350 4050
-Wire Wire Line
-	1350 4050 1350 4250
-Wire Wire Line
-	1350 3850 1450 3850
-Connection ~ 1350 3850
-Wire Wire Line
-	1350 3850 1350 4050
-Wire Wire Line
-	1350 3650 1450 3650
-Connection ~ 1350 3650
-Wire Wire Line
-	1350 3650 1350 3850
-NoConn ~ 2350 2600
-NoConn ~ 4650 1800
-NoConn ~ 4750 1800
-NoConn ~ 4950 1800
-NoConn ~ 5050 1800
-NoConn ~ 5150 1800
+	5150 1150 5150 1800
 NoConn ~ 5750 1800
 NoConn ~ 5850 1800
@@
 P 3650 1250
 F 0 "J9" V 3654 1430 50  0000 L CNN
-F 1 "Conn_02x04_Odd_Even" V 3600 -50 50  0000 L CNN
+F 1 "Conn_02x04_Odd_Even" V 3650 1600 50  0000 L CNN
 F 2 "Connector_PinHeader_2.54mm:PinHeader_2x04_P2.54mm_Vertical" H 3650 1250 50  0001 C CNN
 F 3 "~" H 3650 1250 50  0001 C CNN
@@
 Wire Wire Line
 	4750 6250 7100 6250
-Wire Wire Line
-	2350 2700 2300 2700
-Wire Wire Line
-	2300 2700 2300 2800
-Wire Wire Line
-	2300 2800 2350 2800
-Wire Wire Line
-	2350 2900 2300 2900
-Wire Wire Line
-	2300 2900 2300 3000
-Wire Wire Line
-	2300 3000 2350 3000
 $Comp
 L Device:R_Small R17
@@
 Wire Wire Line
 	5500 7050 5550 7050
+Wire Wire Line
+	1300 3400 2350 3400
+Text GLabel 2100 3200 0    50   BiDi ~ 0
+FIFO_D6
+Text GLabel 2100 3800 0    50   BiDi ~ 0
+FIFO_D2
+Text GLabel 2100 3600 0    50   BiDi ~ 0
+FIFO_D1
+Text GLabel 2100 4200 0    50   Input ~ 0
+FIFO_RXE
+Text GLabel 2100 3000 0    50   Input ~ 0
+FIFO_TXF
+Text GLabel 2100 2700 0    50   Output ~ 0
+FIFO_RDb
+Text GLabel 2100 2600 0    50   Output ~ 0
+FIFO_WRb
+Text GLabel 2100 2800 0    50   Output ~ 0
+FIFO_SIWU
+Text GLabel 2100 2900 0    50   BiDi ~ 0
+FIFO_D3
+Text GLabel 2100 3900 0    50   BiDi ~ 0
+FIFO_D4
+Text GLabel 2100 4300 0    50   BiDi ~ 0
+FIFO_D0
+Wire Wire Line
+	2100 2600 2350 2600
+Wire Wire Line
+	2100 2700 2350 2700
+Wire Wire Line
+	2350 2800 2100 2800
+Wire Wire Line
+	2100 2900 2350 2900
+Wire Wire Line
+	2100 3000 2350 3000
+Wire Wire Line
+	2100 3200 2350 3200
+Wire Wire Line
+	2100 3300 2350 3300
+Wire Wire Line
+	2100 3500 2350 3500
+Wire Wire Line
+	2100 3600 2350 3600
+Wire Wire Line
+	2100 3800 2350 3800
+Wire Wire Line
+	2100 3900 2350 3900
+Wire Wire Line
+	2100 4200 2350 4200
+Wire Wire Line
+	2100 4300 2350 4300
+Wire Wire Line
+	8100 3100 8100 3200
+Wire Wire Line
+	7150 3200 8100 3200
+Wire Wire Line
+	7150 2700 7450 2700
+Wire Wire Line
+	7450 2700 7450 2800
+Wire Wire Line
+	7450 2800 7150 2800
+NoConn ~ 7150 2600
+Text GLabel 2100 3300 0    50   BiDi ~ 0
+FIFO_D5
+Text GLabel 2100 3500 0    50   BiDi ~ 0
+FIFO_D7
+Text GLabel 7600 4000 2    50   Input ~ 0
+ADC_D5
+Text GLabel 7600 3900 2    50   Input ~ 0
+ADC_D4
+Text GLabel 7600 3800 2    50   Input ~ 0
+ADC_D3
+Text GLabel 7600 3700 2    50   Input ~ 0
+ADC_D2
+Text GLabel 7600 3500 2    50   Input ~ 0
+ADC_D1
+Text GLabel 7600 4200 2    50   Input ~ 0
+ADC_D6
+Text GLabel 7600 4300 2    50   Input ~ 0
+ADC_D7
+Text GLabel 7600 3400 2    50   Input ~ 0
+ADC_D0
+Text GLabel 5250 1150 1    50   Input ~ 0
+ADC_DCLK
+Text GLabel 7600 2900 2    50   Input ~ 0
+ADC_DOR
+Text GLabel 4950 1150 1    50   Output ~ 0
+ADC_SYNC
+Wire Wire Line
+	7150 4300 7600 4300
+Wire Wire Line
+	7150 4200 7600 4200
+Wire Wire Line
+	7150 4000 7600 4000
+Wire Wire Line
+	7600 3900 7150 3900
+Wire Wire Line
+	7150 3800 7600 3800
+Wire Wire Line
+	7150 3700 7600 3700
+Wire Wire Line
+	7600 3500 7150 3500
+Wire Wire Line
+	7150 3400 7600 3400
+Wire Wire Line
+	7150 2900 7600 2900
+Wire Wire Line
+	5250 1150 5250 1800
+NoConn ~ 5350 1800
+Wire Wire Line
+	4950 1150 4950 1800
+Text GLabel 4650 1150 1    50   Output ~ 0
+ADC_CSb
+Text GLabel 4750 1150 1    50   Output ~ 0
+ADC_SCLK
+Text GLabel 5050 1150 1    50   BiDi ~ 0
+ADC_SDIO
+$Comp
+L fmc:XC3S50A-VQ100 U5
+U 1 1 60AE5529
+P 1650 3000
+F 0 "U5" H 2800 4100 60  0000 L CNN
+F 1 "XC3S50A-VQ100" H 4350 1800 60  0000 L CNN
+F 2 "Package_QFP:VQFP-100_14x14mm_P0.5mm" H 2500 3650 60  0001 R CNN
+F 3 "" H 2500 3450 60  0001 R CNN
+	1    1650 3000
+	1    0    0    -1
+$EndComp
+Wire Wire Line
+	4650 1150 4650 1800
+Wire Wire Line
+	4750 1150 4750 1800
+Wire Wire Line
+	5050 1150 5050 1800
+NoConn ~ 7150 3100
 $EndSCHEMATC

Commit message: Started to work on analog front-end; ADC connected to fpga
Parts:
- removed J5: GPIO_2V5, Connector_PinHeader_2.54mm:PinHeader_2x08_P2.54mm_Vertical, symbol Connector_Generic:Conn_02x08_Odd_Even
- added J5: GPIO2V5, Connector_PinHeader_2.54mm:PinHeader_2x02_P2.54mm_Vertical, symbol Connector_Generic:Conn_02x02_Odd_Even
Connections:
- net labels added: PGA_CSb, PGA_SCLK, PGA_SDI, PGA_SDO
- wire segments 263 -> 251
- no-connect marks 9 -> 11
Changed lines of the file:
@@
 $Descr A4 11693 8268
 encoding utf-8
-Sheet 3 5
+Sheet 3 7
 Title ""
 Date ""
@@
 	3950 1600 3250 1600
 Wire Wire Line
-	5450 6350 5200 6350
-Wire Wire Line
 	3550 6100 3550 6350
 Connection ~ 3550 6350
@@
 	4050 6100 4050 6450
 $Comp
-L Connector_Generic:Conn_02x08_Odd_Even J5
-U 1 1 608D9FAE
-P 4550 6650
-F 0 "J5" V 4554 7030 50  0000 L CNN
-F 1 "GPIO_2V5" V 5050 6450 50  0000 L CNN
-F 2 "Connector_PinHeader_2.54mm:PinHeader_2x08_P2.54mm_Vertical" H 4550 6650 50  0001 C CNN
-F 3 "~" H 4550 6650 50  0001 C CNN
-	1    4550 6650
-	0    1    1    0
-$EndComp
-Wire Wire Line
-	4350 7050 4350 6950
-Wire Wire Line
-	4350 7050 4550 7050
-Wire Wire Line
-	4550 7050 4550 6950
-Connection ~ 4350 7050
-Wire Wire Line
-	4550 7050 4750 7050
-Wire Wire Line
-	4750 7050 4750 6950
-Connection ~ 4550 7050
-$Comp
 L power:GND #PWR?
 U 1 1 6091690C
@@
 	1    0    0    -1
 $EndComp
-Wire Wire Line
-	4450 6950 4450 7000
-Wire Wire Line
-	4450 7000 4650 7000
-Wire Wire Line
-	4650 6950 4650 7000
-Connection ~ 4650 7000
-Wire Wire Line
-	4650 7000 4850 7000
-Wire Wire Line
-	4850 6950 4850 7000
-Connection ~ 4850 7000
-Wire Wire Line
-	5200 7000 5200 6350
-Connection ~ 5200 6350
-Wire Wire Line
-	5200 6350 3550 6350
 Text GLabel 4550 1150 1    50   Input ~ 0
 FIFO_CLK
@@
 	4550 6400 4650 6400
 Wire Wire Line
-	4650 6400 4650 6450
-Wire Wire Line
 	4650 6100 4650 6300
 Wire Wire Line
 	4650 6300 4750 6300
 Wire Wire Line
-	4750 6300 4750 6450
-Wire Wire Line
 	4150 6950 4150 7050
-Connection ~ 4150 7050
-Wire Wire Line
-	4150 7050 4350 7050
 Wire Wire Line
 	4250 6950 4250 7000
-Wire Wire Line
-	4250 7000 4450 7000
-Connection ~ 4450 7000
-Wire Wire Line
-	4850 7000 5200 7000
 $Comp
 L Device:R_Small R13
@@
 Wire Wire Line
 	5850 7350 5750 7350
-Wire Wire Line
-	4750 7350 4750 7050
-Connection ~ 5450 7350
-Wire Wire Line
-	5450 7350 4750 7350
 Connection ~ 5550 7350
 Wire Wire Line
@@
 Wire Wire Line
 	5750 7350 5650 7350
-Connection ~ 4750 7050
 Wire Wire Line
 	5550 6700 5550 6750
@@
 Wire Wire Line
 	5050 6700 5550 6700
-Wire Wire Line
-	4850 6450 4850 6300
 Wire Wire Line
 	4850 6300 5250 6300
@@
 Text GLabel 7600 3700 2    50   Input ~ 0
 ADC_D2
-Text GLabel 7600 3500 2    50   Input ~ 0
+Text GLabel 7600 3400 2    50   Input ~ 0
 ADC_D1
 Text GLabel 7600 4200 2    50   Input ~ 0
@@
 Text GLabel 7600 4300 2    50   Input ~ 0
 ADC_D7
-Text GLabel 7600 3400 2    50   Input ~ 0
+Text GLabel 7600 2900 2    50   Input ~ 0
 ADC_D0
 Text GLabel 5250 1150 1    50   Input ~ 0
 ADC_DCLK
-Text GLabel 7600 2900 2    50   Input ~ 0
+Text GLabel 7600 3500 2    50   Input ~ 0
 ADC_DOR
 Text GLabel 4950 1150 1    50   Output ~ 0
@@
 	5050 1150 5050 1800
 NoConn ~ 7150 3100
+$Comp
+L Connector_Generic:Conn_02x02_Odd_Even J5
+U 1 1 610A468D
+P 4250 6650
+F 0 "J5" V 4254 6730 50  0000 L CNN
+F 1 "GPIO2V5" V 4345 6730 50  0000 L CNN
+F 2 "Connector_PinHeader_2.54mm:PinHeader_2x02_P2.54mm_Vertical" H 4250 6650 50  0001 C CNN
+F 3 "~" H 4250 6650 50  0001 C CNN
+	1    4250 6650
+	0    1    1    0
+$EndComp
+$Comp
+L power:GND #PWR?
+U 1 1 610A5763
+P 6000 7350
+AR Path="/6086F2E3/610A5763" Ref="#PWR?"  Part="1"
+AR Path="/60AABC24/610A5763" Ref="#PWR?"  Part="1"
+F 0 "#PWR?" H 6000 7100 50  0001 C CNN
+F 1 "GND" H 6005 7177 50  0000 C CNN
+F 2 "" H 6000 7350 50  0001 C CNN
+F 3 "" H 6000 7350 50  0001 C CNN
+	1    6000 7350
+	1    0    0    -1
+$EndComp
+Wire Wire Line
+	5850 7350 6000 7350
+Connection ~ 5850 7350
+Wire Wire Line
+	3550 6350 3650 6350
+Wire Wire Line
+	4250 7000 3650 7000
+Wire Wire Line
+	3650 7000 3650 6350
+Connection ~ 3650 6350
+Wire Wire Line
+	3650 6350 5450 6350
+Text GLabel 4750 7150 3    50   Output ~ 0
+PGA_CSb
+Text GLabel 4650 7150 3    50   Output ~ 0
+PGA_SCLK
+Text GLabel 4550 7150 3    50   Output ~ 0
+PGA_SDI
+Text GLabel 4850 7150 3    50   Input ~ 0
+PGA_SDO
+Wire Wire Line
+	4850 6300 4850 7150
+Wire Wire Line
+	4750 6300 4750 7150
+Wire Wire Line
+	4650 6400 4650 7150
+Wire Wire Line
+	4550 6450 4550 7150
+NoConn ~ 4350 6450
+NoConn ~ 4450 6450
 $EndSCHEMATC

Commit message: more work (don't recall details :-()
Parts:
- J5: footprint Connector_PinHeader_2.54mm:PinHeader_2x02_P2.54mm_Vertical -> Connector_PinHeader_2.54mm:PinHeader_2x03_P2.54mm_Vertical; symbol Connector_Generic:Conn_02x02_Odd_Even -> Connector_Generic:Conn_02x03_Odd_Even
Connections:
- net ADC_CSb: now also U5.86 (IO_L03N_0/GCLK7@Bank@0); no longer U5.89 (IO_L04N_0/GCLK9@Bank@0)
- net ADC_SDIO: now also U5.89 (IO_L04N_0/GCLK9@Bank@0); no longer U5.85 (IO_L03P_0/GCLK6@Bank@0)
- net ADC_SYNC: now also U5.85 (IO_L03P_0/GCLK6@Bank@0); no longer U5.86 (IO_L03N_0/GCLK7@Bank@0)
- net GND: now also J5.1 (Pin_1); no longer J5.4 (Pin_4)
- net PGA_CSb: now also U5.43 (IO_L09P_2/GCLK0@Bank@2); no longer U5.37 (IO_L07N_2/D4@Bank@2)
- net PGA_SCLK: now also U5.37 (IO_L07N_2/D4@Bank@2); no longer U5.36 (IO_L07P_2/D5@Bank@2)
- net PGA_SDI: now also U5.36 (IO_L07P_2/D5@Bank@2); no longer U5.35 (IO_L06N_2/D6@Bank@2)
- net PGA_SDO: now also U5.35 (IO_L06N_2/D6@Bank@2); no longer U5.43 (IO_L09P_2/GCLK0@Bank@2)
- net at U5.32 (IO_L05P_2@Bank@2): now also J5.4 (Pin_4); no longer J5.1 (Pin_1)
- net at U5.33 (IO_L06P_2@Bank@2): now also J5.5 (Pin_5)
- net at U5.34 (IO_L05N_2/D7@Bank@2): now also J5.6 (Pin_6)
- no-connect marks 11 -> 9
Changed lines of the file:
@@
 	3650 7050 3850 7050
 Wire Wire Line
-	3750 6100 3750 6400
-Wire Wire Line
-	3750 6400 4150 6400
-Wire Wire Line
-	4150 6400 4150 6450
-Wire Wire Line
 	4150 6100 4150 6300
 Wire Wire Line
 	4150 6300 4250 6300
 Wire Wire Line
-	4250 6300 4250 6450
-Wire Wire Line
 	4250 6100 4250 6250
 Wire Wire Line
-	4250 6250 4300 6250
-Wire Wire Line
-	4300 6250 4300 6450
-Wire Wire Line
-	4300 6450 4350 6450
-Wire Wire Line
-	4350 6100 4350 6400
-Wire Wire Line
-	4350 6400 4450 6400
-Wire Wire Line
-	4450 6400 4450 6450
-Wire Wire Line
 	4450 6100 4450 6300
 Wire Wire Line
@@
 Wire Wire Line
 	4150 6950 4150 7050
-Wire Wire Line
-	4250 6950 4250 7000
 $Comp
 L Device:R_Small R13
@@
 Text GLabel 7600 3500 2    50   Input ~ 0
 ADC_DOR
-Text GLabel 4950 1150 1    50   Output ~ 0
+Text GLabel 5050 1150 1    50   Output ~ 0
 ADC_SYNC
 Wire Wire Line
@@
 Wire Wire Line
 	4950 1150 4950 1800
-Text GLabel 4650 1150 1    50   Output ~ 0
+Text GLabel 4950 1150 1    50   Output ~ 0
 ADC_CSb
 Text GLabel 4750 1150 1    50   Output ~ 0
 ADC_SCLK
-Text GLabel 5050 1150 1    50   BiDi ~ 0
+Text GLabel 4650 1150 1    50   BiDi ~ 0
 ADC_SDIO
 $Comp
@@
 	5050 1150 5050 1800
 NoConn ~ 7150 3100
-$Comp
-L Connector_Generic:Conn_02x02_Odd_Even J5
-U 1 1 610A468D
-P 4250 6650
-F 0 "J5" V 4254 6730 50  0000 L CNN
-F 1 "GPIO2V5" V 4345 6730 50  0000 L CNN
-F 2 "Connector_PinHeader_2.54mm:PinHeader_2x02_P2.54mm_Vertical" H 4250 6650 50  0001 C CNN
-F 3 "~" H 4250 6650 50  0001 C CNN
-	1    4250 6650
-	0    1    1    0
-$EndComp
 $Comp
 L power:GND #PWR?
@@
 	5850 7350 6000 7350
 Connection ~ 5850 7350
-Wire Wire Line
-	3550 6350 3650 6350
-Wire Wire Line
-	4250 7000 3650 7000
-Wire Wire Line
-	3650 7000 3650 6350
-Connection ~ 3650 6350
-Wire Wire Line
-	3650 6350 5450 6350
+Text GLabel 4850 7150 3    50   Output ~ 0
+PGA_CSb
 Text GLabel 4750 7150 3    50   Output ~ 0
-PGA_CSb
+PGA_SCLK
 Text GLabel 4650 7150 3    50   Output ~ 0
-PGA_SCLK
-Text GLabel 4550 7150 3    50   Output ~ 0
 PGA_SDI
-Text GLabel 4850 7150 3    50   Input ~ 0
+Text GLabel 4550 7150 3    50   Input ~ 0
 PGA_SDO
 Wire Wire Line
@@
 Wire Wire Line
 	4550 6450 4550 7150
-NoConn ~ 4350 6450
-NoConn ~ 4450 6450
+Wire Wire Line
+	3550 6350 4150 6350
+Wire Wire Line
+	4150 6450 4150 6350
+Connection ~ 4150 6350
+Wire Wire Line
+	3750 7000 4250 7000
+Wire Wire Line
+	4250 7000 4250 6950
+Wire Wire Line
+	3750 6100 3750 7000
+Wire Wire Line
+	4450 6950 4350 6950
+Wire Wire Line
+	4250 6300 4250 6450
+Wire Wire Line
+	4150 6350 5450 6350
+$Comp
+L Connector_Generic:Conn_02x03_Odd_Even J5
+U 1 1 610A468D
+P 4250 6750
+F 0 "J5" V 4254 6830 50  0000 L CNN
+F 1 "GPIO2V5" V 3800 6600 50  0000 L CNN
+F 2 "Connector_PinHeader_2.54mm:PinHeader_2x03_P2.54mm_Vertical" H 4250 6750 50  0001 C CNN
+F 3 "~" H 4250 6750 50  0001 C CNN
+	1    4250 6750
+	0    -1   -1   0
+$EndComp
+Wire Wire Line
+	4350 6100 4350 6450
+Wire Wire Line
+	4400 6250 4400 6500
+Wire Wire Line
+	4400 6500 4450 6500
+Wire Wire Line
+	4450 6500 4450 6950
+Wire Wire Line
+	4250 6250 4400 6250
 $EndSCHEMATC
